Commit message: Fixing sigmaban.urdf (dx and dy at 0 for foot_tips

File: Data/sigmaban.urdf (robot description, URDF)
Before this commit: robot metabot, 26 links, 25 joints
Joints:
- joint left_foot_tip: origin xyz=0.01515 0.005 -0.05765 rpy=0 0 0 -> xyz=0 0 -0.05765 rpy=0 0 0
- joint right_foot_tip: origin xyz=0.01515 -0.0055 -0.05765 rpy=0 0 0 -> xyz=0 0 -0.05765 rpy=0 0 0

Commit message: Starting to debug CameraModel based on testModelViewer (not working at all yet)

File: Data/sigmaban.urdf (robot description, URDF)
Before this commit: robot metabot, 26 links, 25 joints
Joints:
- joint camera: origin xyz=0.02277 0 0.068925 rpy=0 0 0 -> xyz=0.02277 0 0.068925 rpy=0 1.5708 0

Commit message: Fixing sigmaban.urdf head rotation

File: Data/sigmaban.urdf (robot description, URDF)
Before this commit: robot metabot, 26 links, 25 joints
Joints:
- joint camera: origin xyz=0.02277 0 0.068925 rpy=0 1.5708 0 -> xyz=0.02277 0 0.068925 rpy=-1.5708 0 -1.5708
