Commit message: Updating the humanoidTest.urdf

File: Data/humanoidTest.urdf (robot description, URDF)
Before this commit: robot metabot, 26 links, 25 joints
Joints:
- joint left_ankle_pitch: origin xyz=0 0 -0.14 rpy=0 0 0 -> xyz=0 0 -0.125 rpy=0 0 0
- joint left_foot_tip: origin xyz=0 0 -0.05765 rpy=0 0 0 -> xyz=0 0 -0.05 rpy=0 0 0
- joint left_hip_yaw: origin xyz=0 0.046375 0 rpy=0 -0 0 -> xyz=0 0.05 0 rpy=0 -0 0
- joint left_knee: origin xyz=0 0 -0.14 rpy=0 0 0 -> xyz=0 0 -0.125 rpy=0 0 0
- joint right_ankle_pitch: origin xyz=0 0 -0.14 rpy=0 0 0 -> xyz=0 0 -0.125 rpy=0 0 0
- joint right_foot_tip: origin xyz=0 0 -0.05765 rpy=0 0 0 -> xyz=0 0 -0.05 rpy=0 0 0
- joint right_hip_yaw: origin xyz=0 -0.046375 0 rpy=0 0 0 -> xyz=0 -0.05 0 rpy=0 0 0
- joint right_knee: origin xyz=0 0 -0.14 rpy=0 0 0 -> xyz=0 0 -0.125 rpy=0 0 0
